Commit message: add yolo_ros2 opncv_ros2

File: install/aurora1/share/aurora1/description/robot.urdf.xacro (robot description, xacro)
@@ -4,5 +4,5 @@
     <!-- <xacro:include filename="gazebo_controller_v2.xacro"/> -->
     <!-- <xacro:include filename="ros2_control_4wd_v2.xacro"/> -->
-    <!-- <xacro:include filename="camera.xacro"/> -->
+    <xacro:include filename="camera.xacro"/>
     <!-- <xacro:include filename="depth_camera.xacro"/> -->
     <xacro:include filename="lidar.xacro"/>

File: install/aurora_drive/share/aurora_drive/description/camera.xacro (robot description, xacro)
@@ -5,5 +5,5 @@
         <parent link="chassis_link"/>
         <child link="camera_link"/>
-        <origin xyz="1.02 0 0" rpy="0 0 0"/>
+        <origin xyz="0.5 0 -0.10" rpy="0 0 0"/>
     </joint>
     <link name="camera_link">
