Commit message: add gps_pkg

File: install/aurora1/share/aurora1/description/camera.xacro (robot description, xacro)
@@ -1 +1,48 @@
-/home/aurora/aurora_sim_v2/build/aurora1/description/camera.xacro
+<?xml version="1.0"?>
+<robot xmlns:xacro="http://ros.org/wiki/xacro" >
+    <!-- Camera Sensor -->
+    <joint name="camera_joint" type="fixed">
+        <parent link="chassis_link"/>
+        <child link="camera_link"/>
+        <origin xyz="1.02 0 0" rpy="0 0 0"/>
+    </joint>
+    <link name="camera_link">
+        <visual>
+            <origin xyz="0 0 0"/>
+            <geometry>
+                <box size="0.01 0.1 0.1"/>
+            </geometry>
+            <material name="red"/>
+        </visual>
+    </link>
+    <joint name="camera_optical_joint" type="fixed">
+        <parent link="camera_link"/>
+        <child link="camera_link_optical"/>
+        <origin xyz="0 0 0" rpy="${-pi/2} 0 ${-pi/2}"/>
+    </joint>
+    <link name="camera_link_optical"></link>
+    <!-- Gazebo properties for Camera sensor -->
+    <gazebo reference="camera_link">
+        <material>Gazebo/Black</material>
+        <sensor name="camera" type="camera">
+            <pose> 0 0 0 0 0 0 </pose>
+            <visualize>true</visualize>
+            <update_rate>20</update_rate>
+            <camera>
+                <horizontal_fov>1.089</horizontal_fov>
+                <image>
+                    <width>640</width>
+                    <height>480</height>
+                    <format>R8G8B8</format>
+                </image>
+                <clip>
+                    <near>0.1</near>
+                    <far>8.0</far>
+                </clip>
+            </camera>
+            <plugin name="camera_controller" filename="libgazebo_ros_camera.so">
+                <frame_name>camera_link_optical</frame_name>
+            </plugin>
+        </sensor>
+    </gazebo>
+</robot>

File: install/aurora1/share/aurora1/description/depth_camera.xacro (robot description, xacro)
@@ -1 +1,48 @@
-/home/aurora/aurora_sim_v2/build/aurora1/description/depth_camera.xacro
+<?xml version="1.0"?>
+<robot xmlns:xacro="http://ros.org/wiki/xacro" >
+    <!-- Camera Sensor -->
+    <joint name="camera_joint" type="fixed">
+        <parent link="chassis_link"/>
+        <child link="camera_link"/>
+        <origin xyz="1.02 0 0" rpy="0 0 0"/>
+    </joint>
+    <link name="camera_link">
+        <visual>
+            <origin xyz="0 0 0"/>
+            <geometry>
+                <box size="0.01 0.1 0.1"/>
+            </geometry>
+            <material name="red"/>
+        </visual>
+    </link>
+    <joint name="camera_optical_joint" type="fixed">
+        <parent link="camera_link"/>
+        <child link="camera_link_optical"/>
+        <origin xyz="0 0 0" rpy="${-pi/2} 0 ${-pi/2}"/>
+    </joint>
+    <link name="camera_link_optical"></link>
+    <!-- Gazebo properties for Camera sensor -->
+    <gazebo reference="camera_link">
+        <material>Gazebo/Black</material>
+        <sensor name="camera" type="depth">
+            <pose> 0 0 0 0 0 0 </pose>
+            <visualize>true</visualize>
+            <update_rate>20</update_rate>
+            <camera>
+                <horizontal_fov>1.089</horizontal_fov>
+                <image>
+                    <width>640</width>
+                    <height>480</height>
+                    <format>R8G8B8</format>
+                </image>
+                <clip>
+                    <near>0.1</near>
+                    <far>8.0</far>
+                </clip>
+            </camera>
+            <plugin name="camera_controller" filename="libgazebo_ros_camera.so">
+                <frame_name>camera_link_optical</frame_name>
+            </plugin>
+        </sensor>
+    </gazebo>
+</robot>

File: install/aurora1/share/aurora1/description/inertial_macros.xacro (robot description, xacro)
@@ -1 +1,32 @@
-/home/aurora/aurora_sim_v2/build/aurora1/description/inertial_macros.xacro
+<?xml version="1.0"?>
+<robot xmlns:xacro="http://www.ros.org/wiki/xacro" >
+    <!-- Specify some standard inertial calculations https://en.wikipedia.org/wiki/List_of_moments_of_inertia -->
+    <!-- These make use of xacro's mathematical functionality -->
+    <!-- <xacro:macro name="inertial_sphere" params="mass radius *origin">
+        <inertial>
+            <xacro:insert_block name="origin"/>
+            <mass value="${mass}" />
+            <inertia ixx="${(2/5) * mass * (radius*radius)}" ixy="0.0" ixz="0.0"
+                    iyy="${(2/5) * mass * (radius*radius)}" iyz="0.0"
+                    izz="${(2/5) * mass * (radius*radius)}" />
+        </inertial>
+    </xacro:macro>   -->
+    <xacro:macro name="inertial_box" params="mass x y z *origin">
+        <inertial>
+            <xacro:insert_block name="origin"/>
+            <mass value="${mass}" />
+            <inertia ixx="${(1/12) * mass * (y*y+z*z)}" ixy="0.0" ixz="0.0"
+                    iyy="${(1/12) * mass * (x*x+z*z)}" iyz="0.0"
+                    izz="${(1/12) * mass * (x*x+y*y)}" />
+        </inertial>
+    </xacro:macro>
+    <xacro:macro name="inertial_cylinder" params="mass length radius *origin">
+        <inertial>
+            <xacro:insert_block name="origin"/>
+            <mass value="${mass}" />
+            <inertia ixx="${(1/12) * mass * (3*radius*radius + length*length)}" ixy="0.0" ixz="0.0"
+                    iyy="${(1/12) * mass * (3*radius*radius + length*length)}" iyz="0.0"
+                    izz="${(1/2) * mass * (radius*radius)}" />
+        </inertial>
+    </xacro:macro>
+</robot>

File: install/aurora1/share/aurora1/description/lidar.xacro (robot description, xacro)
@@ -1 +1,86 @@
-/home/aurora/aurora_sim_v2/build/aurora1/description/lidar.xacro
+<?xml version="1.0"?>
+<robot xmlns:xacro="http://ros.org/wiki/xacro" >
+    <!-- LiDAR Support Post -->
+    <joint name="lidar_post_joint" type="fixed">
+        <parent link="chassis_link"/>
+        <child link="lidar_post"/>
+        <origin xyz="0.3 0 0.1" rpy="0 0 0"/>
+    </joint>
+    <link name="lidar_post">
+        <visual>
+            <origin xyz="0 0 0.075"/>
+            <geometry>
+                <cylinder radius="0.01" length="0.15"/>
+            </geometry>
+            <material name="silver">
+                <color rgba="0.8 0.8 0.8 1"/>
+            </material>
+        </visual>
+        <collision>
+            <origin xyz="0 0 0.075"/>
+            <geometry>
+                <cylinder radius="0.01" length="0.15"/>
+            </geometry>
+        </collision>
+        <xacro:inertial_cylinder mass="0.05" length="0.15" radius="0.01">
+            <origin xyz="0 0 0.075" rpy="0 0 0"/>
+        </xacro:inertial_cylinder>
+    </link>
+    <!-- LiDAR Sensor -->
+    <joint name="laser_joint" type="fixed">
+        <parent link="lidar_post"/>
+        <child link="laser_frame"/>
+        <origin xyz="0 0 0.15" rpy="0 0 0"/>
+    </joint>
+    <link name="laser_frame">
+        <visual>
+            <origin xyz="0 0 0.02"/>
+            <geometry>
+                <cylinder radius="0.05" length="0.04"/>
+            </geometry>
+            <material name="red"/>
+        </visual>
+        <collision>
+            <geometry>
+                <cylinder radius="0.05" length="0.04"/>
+            </geometry>
+            <material name="black"/>
+        </collision>
+        <xacro:inertial_cylinder mass="0.01" length="0.04" radius="0.05">
+            <origin xyz="0 0 0" rpy="0 0 0"/>
+        </xacro:inertial_cylinder>
+    </link>
+    <!-- Gazebo properties for LiDAR post -->
+    <gazebo reference="lidar_post">
+        <material>Gazebo/Grey</material>
+    </gazebo>
+    <!-- Gazebo properties for LiDAR sensor -->
+    <gazebo reference="laser_frame">
+        <material>Gazebo/Black</material>
+        <sensor name="laser" type="ray">
+            <pose> 0 0 0.02 0 0 0 </pose>
+            <visualize>true</visualize>
+            <update_rate>20</update_rate>
+            <ray>
+                <scan>
+                    <horizontal>
+                        <samples>360</samples>
+                        <min_angle>-3.14</min_angle>
+                        <max_angle>3.14</max_angle>
+                    </horizontal>
+                </scan>
+                <range>
+                    <min>0.3</min>
+                    <max>12</max>
+                </range>
+            </ray>
+            <plugin name="laser_controller" filename="libgazebo_ros_ray_sensor.so">
+                <ros>
+                    <argument>~/out:=scan</argument>
+                </ros>
+                <output_type>sensor_msgs/LaserScan</output_type>
+                <frame_name>laser_frame</frame_name>
+            </plugin>
+        </sensor>
+    </gazebo>
+</robot>

File: install/aurora1/share/aurora1/description/robot.urdf.xacro (robot description, xacro)
@@ -1 +1,10 @@
-/home/aurora/aurora_sim_v2/build/aurora1/description/robot.urdf.xacro
+<?xml version="1.0"?>
+<robot xmlns:xacro="http://www.ros.org/wiki/xacro"  name="robot">
+    <xacro:include filename="robot_core_4wd_v2.xacro"/>
+    <!-- <xacro:include filename="gazebo_controller_v2.xacro"/> -->
+    <!-- <xacro:include filename="ros2_control_4wd_v2.xacro"/> -->
+    <!-- <xacro:include filename="camera.xacro"/> -->
+    <!-- <xacro:include filename="depth_camera.xacro"/> -->
+    <xacro:include filename="lidar.xacro"/>
+    <xacro:include filename="ros2_control_4wd_v2.xacro"/>
+</robot>

File: install/aurora1/share/aurora1/description/robot_core_4wd_v2.xacro (robot description, xacro)
@@ -1 +1,259 @@
-/home/aurora/aurora_sim_v2/build/aurora1/description/robot_core_4wd_v2.xacro
+<?xml version="1.0"?>
+<robot xmlns:xacro="http://ros.org/wiki/xacro">
+  <xacro:include filename="inertial_macros.xacro"/>
+  <material name="white">
+    <color rgba="1 1 1 1"/>
+  </material>
+  <material name="black">
+    <color rgba="0 0 0 1"/>
+  </material>
+  <material name="red">
+    <color rgba="1 0 0 1"/>
+  </material>
+  <!-- base link -->
+  <link name="base_link">
+  </link>
+  <!-- base_foot_link-->
+  <joint name="base_foot_joint" type="fixed">
+    <parent link="base_link"/>
+    <child link="base_foot_link"/>
+    <origin xyz="0 0 0" rpy="0 0 0"/>
+  </joint>
+  <link name="base_foot_link">
+  </link>
+  <!--chassis link-->
+  <joint name= "chassis_joint" type="fixed">
+    <parent link="base_link"/>
+    <child link="chassis_link"/>
+    <origin xyz="0 0 0.4" rpy="0 0 0"/>
+  </joint>
+  <link name="chassis_link">
+    <visual>
+      <origin xyz ="0 0 0"/>
+      <geometry>
+        <box size="1.0 0.8 0.3"/>
+      </geometry>
+      <material name="white"/>
+    </visual>
+    <collision>
+      <origin xyz ="0 0 0"/>
+      <geometry>
+        <box size="1.0 0.8 0.3"/>
+      </geometry>
+    </collision>
+    <xacro:inertial_box mass="3.0" x="1.0" y="0.8" z="0.3">
+      <origin xyz="0 0 0" rpy="0 0 0"/>
+    </xacro:inertial_box>
+  </link>
+  <gazebo reference="chassis_link">
+    <material>Gazebo/White</material>
+  </gazebo>
+  <!-- left_front_steering-->
+  <joint name="left_front_steering_joint" type="continuous">
+    <parent link="chassis_link"/>
+    <child link="left_front_steering_link"/>
+    <origin xyz="0.5 0.4 -0.15" rpy="0 0 0"/>
+    <axis xyz="0 0 1"/>
+  </joint>
+  <link name="left_front_steering_link">
+    <visual>
+      <geometry>
+        <cylinder radius="0.1" length="0.3"/>
+      </geometry>
+      <material name="black"/>
+    </visual>
+    <collision>
+      <geometry>
+        <cylinder radius="0.1" length="0.3"/>
+      </geometry>
+    </collision>
+    <xacro:inertial_cylinder mass="0.25" length="0.3" radius="0.1">
+      <origin xyz="0 0 0" rpy="0 0 0"/>
+    </xacro:inertial_cylinder>
+  </link>
+  <gazebo reference="left_front_steering_link">
+    <material>Gazebo/Red</material>
+  </gazebo>
+<!-- left_front_wheel-->
+  <joint name="left_front_wheel_joint" type="continuous">
+    <parent link="left_front_steering_link"/>
+    <child link="left_front_wheel_link"/>
+    <origin xyz="0 0 -0.15" rpy="${-pi/2} 0 0"/>
+    <axis xyz="0 0 1"/>
+  </joint>
+  <link name="left_front_wheel_link">
+    <visual>
+      <geometry>
+        <cylinder radius ="0.15" length="0.2"/>
+      </geometry>
+      <material name="black"/>
+    </visual>
+    <collision>
+      <geometry>
+        <cylinder radius ="0.15" length="0.2"/>
+      </geometry>
+    </collision>
+    <xacro:inertial_cylinder mass="0.5" length="0.2" radius="0.15">
+      <origin xyz="0 0 0" rpy="0 0 0"/>
+    </xacro:inertial_cylinder>
+  </link>
+  <gazebo reference="left_front_wheel_link">
+    <material>Gazebo/Black</material>
+  </gazebo>
+  <!-- right_front_steering-->
+  <joint name="right_front_steering_joint" type="continuous">
+    <parent link="chassis_link"/>
+    <child link="right_front_steering_link"/>
+    <origin xyz="0.5 -0.4 -0.15" rpy="0 0 0"/>
+    <axis xyz="0 0 1"/>
+  </joint>
+  <link name="right_front_steering_link">
+    <visual>
+      <geometry>
+        <cylinder radius="0.1" length="0.3"/>
+      </geometry>
+      <material name="black"/>
+    </visual>
+    <collision>
+      <geometry>
+        <cylinder radius="0.1" length="0.3"/>
+      </geometry>
+    </collision>
+    <xacro:inertial_cylinder mass="0.25" length="0.3" radius="0.1">
+      <origin xyz="0 0 0" rpy="0 0 0"/>
+    </xacro:inertial_cylinder>
+  </link>
+  <gazebo reference="right_front_steering_link">
+    <material>Gazebo/Red</material>
+  </gazebo>
+<!-- right_front_wheel-->
+  <joint name="right_front_wheel_joint" type="continuous">
+    <parent link="right_front_steering_link"/>
+    <child link="right_front_wheel_link"/>
+    <origin xyz="0 0 -0.15" rpy="${-pi/2} 0 0"/>
+    <axis xyz="0 0 1"/>
+  </joint>
+  <link name="right_front_wheel_link">
+    <visual>
+      <geometry>
+        <cylinder radius ="0.15" length="0.2"/>
+      </geometry>
+      <material name="black"/>
+    </visual>
+    <collision>
+      <geometry>
+        <cylinder radius ="0.15" length="0.2"/>
+      </geometry>
+    </collision>
+    <xacro:inertial_cylinder mass="0.5" length="0.2" radius="0.15">
+      <origin xyz="0 0 0" rpy="0 0 0"/>
+    </xacro:inertial_cylinder>
+  </link>
+  <gazebo reference="right_front_wheel_link">
+    <material>Gazebo/Black</material>
+  </gazebo>
+  <!-- left_back_steering-->
+  <joint name="left_back_steering_joint" type="continuous">
+    <parent link="chassis_link"/>
+    <child link="left_back_steering_link"/>
+    <origin xyz="-0.5 0.4 -0.15" rpy="0 0 0"/>
+    <axis xyz="0 0 1"/>
+  </joint>
+  <link name="left_back_steering_link">
+    <visual>
+      <geometry>
+        <cylinder radius="0.1" length="0.3"/>
+      </geometry>
+      <material name="black"/>
+    </visual>
+    <collision>
+      <geometry>
+        <cylinder radius="0.1" length="0.3"/>
+      </geometry>
+    </collision>
+    <xacro:inertial_cylinder mass="0.25" length="0.3" radius="0.1">
+      <origin xyz="0 0 0" rpy="0 0 0"/>
+    </xacro:inertial_cylinder>
+  </link>
+  <gazebo reference="left_back_steering_link">
+    <material>Gazebo/Red</material>
+  </gazebo>
+<!-- left_back_wheel-->
+  <joint name="left_back_wheel_joint" type="continuous">
+    <parent link="left_back_steering_link"/>
+    <child link="left_back_wheel_link"/>
+    <origin xyz="0 0 -0.15" rpy="${-pi/2} 0 0"/>
+    <axis xyz="0 0 1"/>
+  </joint>
+  <link name="left_back_wheel_link">
+    <visual>
+      <geometry>
+        <cylinder radius ="0.15" length="0.2"/>
+      </geometry>
+      <material name="black"/>
+    </visual>
+    <collision>
+      <geometry>
+        <cylinder radius ="0.15" length="0.2"/>
+      </geometry>
+    </collision>
+    <xacro:inertial_cylinder mass="0.5" length="0.2" radius="0.15">
+      <origin xyz="0 0 0" rpy="0 0 0"/>
+    </xacro:inertial_cylinder>
+  </link>
+  <gazebo reference="left_back_wheel_link">
+    <material>Gazebo/Black</material>
+  </gazebo>
+  <!-- right_back_steering-->
+  <joint name="right_back_steering_joint" type="continuous">
+    <parent link="chassis_link"/>
+    <child link="right_back_steering_link"/>
+    <origin xyz="-0.5 -0.4 -0.15" rpy="0 0 0"/>
+    <axis xyz="0 0 1"/>
+  </joint>
+  <link name="right_back_steering_link">
+    <visual>
+      <geometry>
+        <cylinder radius="0.1" length="0.3"/>
+      </geometry>
+      <material name="black"/>
+    </visual>
+    <collision>
+      <geometry>
+        <cylinder radius="0.1" length="0.3"/>
+      </geometry>
+    </collision>
+    <xacro:inertial_cylinder mass="0.25" length="0.3" radius="0.1">
+      <origin xyz="0 0 0" rpy="0 0 0"/>
+    </xacro:inertial_cylinder>
+  </link>
+  <gazebo reference="right_back_steering_link">
+    <material>Gazebo/Red</material>
+  </gazebo>
+<!-- right_back_wheel-->
+  <joint name="right_back_wheel_joint" type="continuous">
+    <parent link="right_back_steering_link"/>
+    <child link="right_back_wheel_link"/>
+    <origin xyz="0 0 -0.15" rpy="${-pi/2} 0 0"/>
+    <axis xyz="0 0 1"/>
+  </joint>
+  <link name="right_back_wheel_link">
+    <visual>
+      <geometry>
+        <cylinder radius ="0.15" length="0.2"/>
+      </geometry>
+      <material name="black"/>
+    </visual>
+    <collision>
+      <geometry>
+        <cylinder radius ="0.15" length="0.2"/>
+      </geometry>
+    </collision>
+    <xacro:inertial_cylinder mass="0.5" length="0.2" radius="0.15">
+      <origin xyz="0 0 0" rpy="0 0 0"/>
+    </xacro:inertial_cylinder>
+  </link>
+  <gazebo reference="right_back_wheel_link">
+    <material>Gazebo/Black</material>
+  </gazebo>
+</robot>

File: install/aurora1/share/aurora1/description/ros2_control_4wd_v2.xacro (robot description, xacro)
@@ -1 +1,53 @@
-/home/aurora/aurora_sim_v2/build/aurora1/description/ros2_control_4wd_v2.xacro
+<?xml version="1.0"?>
+<robot xmlns:xacro="http://www.ros.org/wiki/xacro">
+  <ros2_control name="GazeboSystem" type="system">
+    <hardware>
+      <plugin>gazebo_ros2_control/GazeboSystem</plugin>
+    </hardware>
+    <!-- 後輪駆動 -->
+    <joint name="left_back_wheel_joint">
+      <command_interface name="velocity"/>
+      <state_interface name="velocity"/>
+      <state_interface name="position"/>
+    </joint>
+    <joint name="right_back_wheel_joint">
+      <command_interface name="velocity"/>
+      <state_interface name="velocity"/>
+      <state_interface name="position"/>
+    </joint>
+    <!-- 前輪駆動 -->
+    <joint name="left_front_wheel_joint">
+      <command_interface name="velocity"/>
+      <state_interface name="velocity"/>
+      <state_interface name="position"/>
+    </joint>
+    <joint name="right_front_wheel_joint">
+      <command_interface name="velocity"/>
+      <state_interface name="velocity"/>
+      <state_interface name="position"/>
+    </joint>
+    <!-- 前輪ステアリング -->
+    <joint name="left_front_steering_joint">
+      <command_interface name="position"/>
+      <state_interface name="position"/>
+    </joint>
+    <joint name="right_front_steering_joint">
+      <command_interface name="position"/>
+      <state_interface name="position"/>
+    </joint>
+    <!-- 後輪ステアリング -->
+    <joint name="left_back_steering_joint">
+      <command_interface name="position"/>
+      <state_interface name="position"/>
+    </joint>
+    <joint name="right_back_steering_joint">
+      <command_interface name="position"/>
+      <state_interface name="position"/>
+    </joint>
+  </ros2_control>
+  <gazebo>
+    <plugin name="gazebo_ros2_control" filename="libgazebo_ros2_control.so">
+      <parameters>$(find aurora1)/config/rover_controller_4wd_v2.yaml</parameters>
+    </plugin>
+  </gazebo>
+</robot>

File: install/aurora_drive/share/aurora_drive/description/camera.xacro (robot description, xacro)
@@ -1 +1,48 @@
-/home/aurora/aurora_sim_v2/build/aurora_drive/description/camera.xacro
+<?xml version="1.0"?>
+<robot xmlns:xacro="http://ros.org/wiki/xacro" >
+    <!-- Camera Sensor -->
+    <joint name="camera_joint" type="fixed">
+        <parent link="chassis_link"/>
+        <child link="camera_link"/>
+        <origin xyz="1.02 0 0" rpy="0 0 0"/>
+    </joint>
+    <link name="camera_link">
+        <visual>
+            <origin xyz="0 0 0"/>
+            <geometry>
+                <box size="0.01 0.1 0.1"/>
+            </geometry>
+            <material name="red"/>
+        </visual>
+    </link>
+    <joint name="camera_optical_joint" type="fixed">
+        <parent link="camera_link"/>
+        <child link="camera_link_optical"/>
+        <origin xyz="0 0 0" rpy="${-pi/2} 0 ${-pi/2}"/>
+    </joint>
+    <link name="camera_link_optical"></link>
+    <!-- Gazebo properties for Camera sensor -->
+    <gazebo reference="camera_link">
+        <material>Gazebo/Black</material>
+        <sensor name="camera" type="camera">
+            <pose> 0 0 0 0 0 0 </pose>
+            <visualize>true</visualize>
+            <update_rate>20</update_rate>
+            <camera>
+                <horizontal_fov>1.089</horizontal_fov>
+                <image>
+                    <width>640</width>
+                    <height>480</height>
+                    <format>R8G8B8</format>
+                </image>
+                <clip>
+                    <near>0.1</near>
+                    <far>8.0</far>
+                </clip>
+            </camera>
+            <plugin name="camera_controller" filename="libgazebo_ros_camera.so">
+                <frame_name>camera_link_optical</frame_name>
+            </plugin>
+        </sensor>
+    </gazebo>
+</robot>
